File: blahblahVCA.sch (EAGLE design)
At the start: 31 parts, among them IC1 CA3080D, IC2 RC4558D, IC3 CA3130D, Q1 BCM847DS

Commit message: Add files via upload
Parts:
- IC1: value CA3080D -> AS3080D; device wb-ota:CA3080D -> wb-ota:AS3080D
- renumbered C5 to C4
