File: blahblahVCA.MB.brd (EAGLE design)
At the start: 19.7 x 82.9 mm, 31 parts, among them IC1 AS3080D, IC2 RC4558D, IC3 CA3130D, Q1 BCM847DS

Commit message: Add files via upload
Routing:
- net +12V: track 87.1 -> 86.1 mm
Changed lines of the file:
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@@
 <wire x1="19.6725" y1="82.8575" x2="0" y2="82.8575" width="0" layer="20"/>
 <wire x1="0" y1="82.8575" x2="0" y2="0" width="0" layer="20"/>
-<dimension x1="2.06375" y1="78.74" x2="2.06375" y2="16.51" x3="-0.9525" y3="47.625" textsize="1.778" layer="20"/>
-<dimension x1="2.06375" y1="78.74" x2="14.76375" y2="78.74" x3="8.41375" y3="83.82" textsize="1.778" layer="20"/>
-<dimension x1="0" y1="82.8575" x2="19.6725" y2="82.8575" x3="9.83625" y3="87.63" textsize="1.778" layer="20"/>
-<dimension x1="0" y1="82.8575" x2="0" y2="0" x3="-5.08" y3="41.42875" textsize="1.778" layer="20"/>
+<dimension x1="2.06375" y1="78.74" x2="2.06375" y2="16.51" x3="-0.9525" y3="47.625" textsize="1.778" layer="49"/>
+<dimension x1="2.06375" y1="78.74" x2="14.76375" y2="78.74" x3="8.41375" y3="83.82" textsize="1.778" layer="48"/>
+<dimension x1="0" y1="82.8575" x2="19.6725" y2="82.8575" x3="9.83625" y3="87.63" textsize="1.778" layer="48"/>
+<dimension x1="0" y1="82.8575" x2="0" y2="0" x3="-5.08" y3="41.42875" textsize="1.778" layer="48"/>
 </plain>
 <attributes>
@@
 </element>
 <element name="R5" library="wb-rcl" package="R1206" value="100k" x="3.33375" y="58.42" smashed="yes" rot="MR0">
-<attribute name="NAME" x="7.14375" y="59.69" size="1.27" layer="26" rot="MR270"/>
+<attribute name="NAME" x="3.81" y="60.96" size="1.27" layer="26" rot="MR180"/>
 </element>
 <element name="R6" library="wb-rcl" package="R1206" value="100k" x="7.14375" y="48.26" smashed="yes" rot="MR180">
-<attribute name="NAME" x="10.95375" y="49.53" size="1.27" layer="26" rot="MR270"/>
+<attribute name="NAME" x="7.62" y="50.8" size="1.27" layer="26" rot="MR180"/>
 </element>
 <element name="R7" library="wb-rcl" package="R1206" value="75k" x="14.12875" y="48.26" smashed="yes" rot="R270">
@@
 <vertex x="0.47625" y="80.48625"/>
 </polygon>
-<wire x1="9.68375" y1="78.74" x2="2.06375" y2="78.74" width="0" layer="19" extent="1-1"/>
-<wire x1="2.06375" y1="16.51" x2="7.14375" y2="11.43" width="0" layer="19" extent="1-1"/>
 </signal>
 <signal name="N$2">
@@
 <wire x1="12.22375" y1="44.45" x2="16.03375" y2="44.45" width="0.4064" layer="16"/>
 <wire x1="4.60375" y1="2.54" x2="4.60375" y2="5.08" width="0.4064" layer="16"/>
-<wire x1="9.68375" y1="34.29" x2="13.49375" y2="38.1" width="0.4064" layer="16"/>
-<wire x1="13.49375" y1="38.1" x2="16.03375" y2="38.1" width="0.4064" layer="16"/>
 <via x="16.03375" y="38.1" extent="1-16" drill="0.6" diameter="0.6"/>
 <wire x1="16.03375" y1="41.275" x2="16.03375" y2="38.1" width="0.4064" layer="1"/>
@@
 <wire x1="18.57375" y1="15.24" x2="18.57375" y2="35.56" width="0.4064" layer="1"/>
 <wire x1="7.14375" y1="13.97" x2="17.30375" y2="13.97" width="0.4064" layer="16"/>
+<wire x1="9.68375" y1="36.678" x2="14.61175" y2="36.678" width="0.4064" layer="16"/>
+<wire x1="14.61175" y1="36.678" x2="16.03375" y2="38.1" width="0.4064" layer="16"/>
 </signal>
 <signal name="-12V">
